File: hardware/kicad/pipod-carrier/pipod-carrier.kicad_sch (KiCad schematic)
At the start: 23 parts, among them J1 Raspberry_Pi_Zero_2W, J3 Conn_02x06_Odd_Even, J5 Conn_01x02, SW1 Volume Up, SW2 Volume Down, U1 Adafruit Seesaw Encoder, U2 Adafruit 2.2 PiTFT HAT - 320x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, U3 PCM5102A, U4 TPA6132

Commit message: Initial PCB layout complete
Parts:
- removed TP7: TP_TFT_3V3, TestPoint:TestPoint_Plated_Hole_D2.0mm, symbol Connector:TestPoint
- removed TP8: TP_SEESAW_3V3, TestPoint:TestPoint_Plated_Hole_D2.0mm, symbol Connector:TestPoint
Changed lines of the file:
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@@
 	)
 	(junction
-		(at 93.98 80.01)
-		(diameter 0)
-		(color 0 0 0 0)
-	)
-	(junction
 		(at 134.62 35.56)
 		(diameter 0)
@@
 	)
 	(junction
-		(at 102.87 102.87)
-		(diameter 0)
-		(color 0 0 0 0)
-	)
-	(junction
 		(at 107.95 105.41)
 		(diameter 0)
@@
 	(wire
 		(pts
-			(xy 93.98 80.01) (xy 93.98 90.17)
-		)
-		(stroke
-			(width 0)
-			(type default)
-		)
-	)
-	(wire
-		(pts
 			(xy 105.41 102.87) (xy 105.41 111.76)
 		)
@@
 	(wire
 		(pts
-			(xy 78.74 91.44) (xy 78.74 93.98)
-		)
-		(stroke
-			(width 0)
-			(type default)
-		)
-	)
-	(wire
-		(pts
 			(xy 153.67 134.62) (xy 153.67 147.32)
 		)
@@
 	(wire
 		(pts
-			(xy 90.17 72.39) (xy 90.17 80.01)
-		)
-		(stroke
-			(width 0)
-			(type default)
-		)
-	)
-	(wire
-		(pts
 			(xy 124.46 104.14) (xy 118.11 104.14)
 		)
@@
 	(wire
 		(pts
-			(xy 97.79 102.87) (xy 102.87 102.87)
-		)
-		(stroke
-			(width 0)
-			(type default)
-		)
-	)
-	(wire
-		(pts
 			(xy 121.92 132.08) (xy 118.11 132.08)
 		)
@@
 	(wire
 		(pts
-			(xy 90.17 80.01) (xy 93.98 80.01)
-		)
-		(stroke
-			(width 0)
-			(type default)
-		)
-	)
-	(wire
-		(pts
 			(xy 55.88 41.91) (xy 127 41.91)
 		)
@@
 	(wire
 		(pts
-			(xy 102.87 102.87) (xy 105.41 102.87)
+			(xy 97.79 102.87) (xy 105.41 102.87)
 		)
 		(stroke
@@
 	(wire
 		(pts
-			(xy 78.74 93.98) (xy 102.87 93.98)
-		)
-		(stroke
-			(width 0)
-			(type default)
-		)
-	)
-	(wire
-		(pts
 			(xy 158.75 116.84) (xy 152.4 116.84)
 		)
@@
 	(wire
 		(pts
-			(xy 102.87 93.98) (xy 102.87 102.87)
-		)
-		(stroke
-			(width 0)
-			(type default)
-		)
-	)
-	(wire
-		(pts
 			(xy 182.88 82.55) (xy 232.41 82.55)
 		)
@@
 	(wire
 		(pts
-			(xy 93.98 74.93) (xy 93.98 80.01)
+			(xy 93.98 74.93) (xy 93.98 90.17)
 		)
 		(stroke
@@
 	)
 	(symbol
-		(lib_id "Connector:TestPoint")
-		(at 90.17 72.39 0)
-		(unit 1)
-		(body_style 1)
-		(exclude_from_sim no)
-		(in_bom yes)
-		(on_board yes)
-		(in_pos_files yes)
-		(dnp no)
-		(property "Reference" "TP7"
-			(at 83.82 69.088 0)
-			(show_name no)
-			(do_not_autoplace no)
-			(effects
-				(font
-					(size 0.762 0.762)
-				)
-				(justify left)
-			)
-		)
-		(property "Value" "TP_TFT_3V3"
-			(at 80.772 70.612 0)
-			(show_name no)
-			(do_not_autoplace no)
-			(effects
-				(font
-					(size 0.762 0.762)
-				)
-				(justify left)
-			)
-		)
-		(property "Footprint" "TestPoint:TestPoint_Plated_Hole_D2.0mm"
-			(at 95.25 72.39 0)
-			(hide yes)
-			(show_name no)
-			(do_not_autoplace no)
-			(effects
-				(font
-					(size 1.27 1.27)
-				)
-			)
-		)
-		(property "Datasheet" ""
-			(at 95.25 72.39 0)
-			(hide yes)
-			(show_name no)
-			(do_not_autoplace no)
-			(effects
-				(font
-					(size 1.27 1.27)
-				)
-			)
-		)
-		(property "Description" "test point"
-			(at 90.17 72.39 0)
-			(hide yes)
-			(show_name no)
-			(do_not_autoplace no)
-			(effects
-				(font
-					(size 1.27 1.27)
-				)
-			)
-		)
-		(pin "1"
-		)
-		(instances
-			(project "pipod-carrier"
-				(path "/7155fab1-9c9a-41b5-92ad-f730b415b976"
-					(reference "TP7")
-					(unit 1)
-				)
-			)
-		)
-	)
-	(symbol
 		(lib_id "Connector_Generic:Conn_02x06_Odd_Even")
 		(at 86.36 27.94 0)
@@
 					(unit 1)
 				)
-			)
-		)
-	)
-	(symbol
-		(lib_id "Connector:TestPoint")
-		(at 78.74 91.44 0)
-		(unit 1)
-		(body_style 1)
-		(exclude_from_sim no)
-		(in_bom yes)
-		(on_board yes)
-		(in_pos_files yes)
-		(dnp no)
-		(property "Reference" "TP8"
-			(at 80.518 87.63 0)
-			(show_name no)
-			(do_not_autoplace no)
-			(effects
-				(font
-					(size 0.762 0.762)
-				)
-				(justify left)
-			)
-		)
-		(property "Value" "TP_SEESAW_3V3"
-			(at 80.264 89.154 0)
-			(show_name no)
-			(do_not_autoplace no)
-			(effects
-				(font
-					(size 0.762 0.762)
-				)
-				(justify left)
-			)
-		)
-		(property "Footprint" "TestPoint:TestPoint_Plated_Hole_D2.0mm"
-			(at 83.82 91.44 0)
-			(hide yes)
-			(show_name no)
-			(do_not_autoplace no)
-			(effects
-				(font
-					(size 1.27 1.27)
-				)
-			)
-		)
-		(property "Datasheet" ""
-			(at 83.82 91.44 0)
-			(hide yes)
-			(show_name no)
-			(do_not_autoplace no)
-			(effects
-				(font
-					(size 1.27 1.27)
-				)
-			)
-		)
-		(property "Description" "test point"
-			(at 78.74 91.44 0)
-			(hide yes)
-			(show_name no)
-			(do_not_autoplace no)
-			(effects
-				(font
-					(size 1.27 1.27)
-				)
-			)
-		)
-		(pin "1"
-		)
-		(instances
-			(project "pipod-carrier"
-				(path "/7155fab1-9c9a-41b5-92ad-f730b415b976"
-					(reference "TP8")
-					(unit 1)
-				)
