File: hardware/kicad/pipod-carrier-v2/pipod-carrier-v2.kicad_pcb (KiCad board)
At the start: 2 copper layers, 65 x 110 mm, 16 parts, among them J1 Raspberry_Pi_Zero_2W, J3 Conn_02x06_Odd_Even, J5 Conn_01x02, SW1 Volume Up, SW2 Volume Down, SW3 PWR, U1 Adafruit Seesaw Encoder, U3 PCM5102A, U4 TPA6132

Commit message: added battery slot, relocated display and encoder connectors
Parts:
- added Battery Slot: Battery Slot, pipod_footprints:Battery_Slot, F.Cu at (111.9, 70.6)
- moved U1 26.0 mm to (119.0, 135.2)
- moved J5 13.4 mm to (108.4, 95.4), turned to 180 degrees
- moved TP4 0.66 mm to (115.3, 92.9)
Connections:
- J3 pad 12: unconnected-(J3-Pin_12-Pad12) -> GND
Routing:
- net Net-(J1-GPIO2_/_SDA1): track 75.3 -> 40.9 mm
- net Net-(J1-GPIO3_/_SCL1): track 41.0 -> 25.6 mm
- net /3V3: track 221.1 -> 208.2 mm, vias 5 -> 6
- net /TFT_CE1: track 67.5 -> 70.7 mm
Other:
- board text added: "3V3"
- board text added: "5V"
- board text added: "Audio DAC"
- board text added: "DO NOT MOUNT PI ON THIS SIDE"
- board text added: "Display"
- board text added: "Display 3V3"
- board text added: "GND"
- board text added: "Headphone Amp"
- board text added: "Mount Pi on this Side"
- board text added: "Power"
- board text added: "Raspberry Pi Audio Player v0.1"
- board text added: "Rotary Encoder"
