File: hardware/kicad/pipod-carrier-v2/pipod-carrier-v2.kicad_sch (KiCad schematic)
At the start: 22 parts, among them J1 Raspberry_Pi_Zero_2W, J3 Conn_02x06_Odd_Even, J5 Conn_01x02, SW1 Volume Up, SW2 Volume Down, SW3 PWR, U1 Adafruit Seesaw Encoder, U2 Adafruit 2.2 PiTFT HAT - 320x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, U3 PCM5102A, U4 TPA6132

Commit message: PCB first draft with no errors and updated component placement
Parts:
- removed TP1: TP_TFT_CE1, TestPoint:TestPoint_Plated_Hole_D2.0mm, symbol Connector:TestPoint
- removed TP10: TP_I2C_SCL, TestPoint:TestPoint_Plated_Hole_D2.0mm, symbol Connector:TestPoint
- removed TP11: TP_TFT_CE0, TestPoint:TestPoint_Plated_Hole_D2.0mm, symbol Connector:TestPoint
- removed TP12: TP_TFT_SCLK, TestPoint:TestPoint_Plated_Hole_D2.0mm, symbol Connector:TestPoint
- removed TP13: TP_TFT_MOSI, TestPoint:TestPoint_Plated_Hole_D2.0mm, symbol Connector:TestPoint
- removed TP14: TP_TFT_DC, TestPoint:TestPoint_Plated_Hole_D2.0mm, symbol Connector:TestPoint
- removed TP15: TP_TFT_MISO, TestPoint:TestPoint_Plated_Hole_D2.0mm, symbol Connector:TestPoint
- removed TP6: TP_TFT_5V, TestPoint:TestPoint_Plated_Hole_D2.0mm, symbol Connector:TestPoint
- removed TP9: TP_I2C_SDA, TestPoint:TestPoint_Plated_Hole_D2.0mm, symbol Connector:TestPoint

Commit message: added battery slot, relocated display and encoder connectors
Connections:
- net GND: now also J3.12 (Pin_12), U2.29 (GND)
- no-connect marks 35 -> 33
Changed lines of the file:
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@@
+	)
+	(junction
+		(at 115.57 87.63)
+		(diameter 0)
+		(color 0 0 0 0)
 	)
 	(junction
@@
 	)
 	(junction
+		(at 172.72 55.88)
+		(diameter 0)
+		(color 0 0 0 0)
+	)
+	(junction
 		(at 139.7 55.88)
 		(diameter 0)
@@
 	)
 	(no_connect
-		(at 93.98 35.56)
-	)
-	(no_connect
 		(at 240.03 59.69)
 	)
@@
 	)
 	(no_connect
-		(at 172.72 55.88)
-	)
-	(no_connect
 		(at 121.92 149.86)
 	)
@@
 	(wire
 		(pts
+			(xy 93.98 35.56) (xy 95.25 35.56)
+		)
+		(stroke
+			(width 0)
+			(type default)
+		)
+	)
+	(wire
+		(pts
 			(xy 97.79 107.95) (xy 107.95 107.95)
 		)
@@
 	(wire
 		(pts
+			(xy 172.72 55.88) (xy 172.72 87.63)
+		)
+		(stroke
+			(width 0)
+			(type default)
+		)
+	)
+	(wire
+		(pts
 			(xy 257.81 129.54) (xy 257.81 40.64)
 		)
@@
 	(wire
 		(pts
+			(xy 172.72 55.88) (xy 173.99 55.88)
+		)
+		(stroke
+			(width 0)
+			(type default)
+		)
+	)
+	(wire
+		(pts
 			(xy 152.4 132.08) (xy 180.34 132.08)
 		)
@@
 		(pts
 			(xy 93.98 74.93) (xy 93.98 90.17)
+		)
+		(stroke
+			(width 0)
+			(type default)
+		)
+	)
+	(wire
+		(pts
+			(xy 115.57 87.63) (xy 172.72 87.63)
 		)
 		(stroke
@@
 		)
 	)
-	(label "TFT_DC"
-		(at 129.54 72.39 0)
+	(label "GND"
+		(at 95.25 35.56 0)
 		(effects
 			(font
@@
 		)
 	)
-	(label "GND"
-		(at 101.6 83.82 0)
+	(label "TFT_DC"
+		(at 129.54 72.39 0)
 		(effects
 			(font
@@
 		)
 	)
-	(label "TFT_BTN3"
-		(at 74.93 27.94 0)
+	(label "GND"
+		(at 101.6 83.82 0)
 		(effects
 			(font
@@
 		)
 	)
+	(label "TFT_BTN3"
+		(at 74.93 27.94 0)
+		(effects
+			(font
+				(size 0.762 0.762)
+			)
+			(justify left bottom)
+		)
+	)
 	(label "GND"
 		(at 35.56 25.4 0)
 		(effects
 			(font
+				(size 0.762 0.762)
+			)
+			(justify left bottom)
+		)
+	)
+	(label "GND"
+		(at 173.99 55.88 0)
+		(effects
+			(font

Commit message: fixed CE0 and CE1 and button 2 and button 4 labels
Connections:
- net TFT_BTN2: now also J1.15 (GPIO22), U2.12 (GPIO_22_BTN2); no longer J1.13 (GPIO27), U2.11 (GPIO_27_BTN4)
- net TFT_BTN4: now also J1.13 (GPIO27), U2.11 (GPIO_27_BTN4); no longer J1.15 (GPIO22), U2.12 (GPIO_22_BTN2)
- net TFT_CE0: now also J1.24 (GPIO8_/_CE0), U2.19 (CE0); no longer J1.26 (GPIO7_/_CE1), U2.20 (CE1)
- net TFT_CE1: now also J1.26 (GPIO7_/_CE1), U2.20 (CE1); no longer J1.24 (GPIO8_/_CE0), U2.19 (CE0)
Changed lines of the file:
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@@
 		)
 	)
-	(label "TFT_CE0"
+	(label "TFT_CE1"
 		(at 148.59 72.39 0)
 		(effects
@@
 		)
 	)
-	(label "TFT_BTN4"
+	(label "TFT_BTN2"
 		(at 119.38 74.93 0)
 		(effects
@@
 		)
 	)
-	(label "TFT_CE1"
+	(label "TFT_CE0"
 		(at 146.05 74.93 0)
 		(effects
@@
 		)
 	)
-	(label "TFT_BTN2"
+	(label "TFT_BTN4"
 		(at 116.84 72.39 0)
 		(effects
